Commit message: Add files via upload
assembly of model

File: src/husky/urdf/teste.xacro (robot description, xacro)
@@ -5,8 +5,8 @@
   <!-- Insert customization below, sample provided: -->
     <xacro:include filename="$(find velodyne_description)/urdf/VLP-16.urdf.xacro"/>
-    <VLP-16 parent="top_plate_link" name="velodyne" topic="/velodyne_points" hz="10" samples="440" gpu="${gpu}">
-    <origin xyz="0 0 0.4" rpy="0 0 0" />
+    <VLP-16 parent="base" name="velodyne" topic="/velodyne_points" hz="10" samples="440" gpu="${gpu}">
+    <origin xyz="0 0 0.1" rpy="0 0 0" />
   </VLP-16>
- <link name="bowler_link">
+ <!-- <link name="bowler_link">
     <visual>
       <geometry>
@@ -20,9 +20,36 @@
       </geometry>
     </collision>
-  </link>
-  <joint name="bowler_joint" type="fixed">
+  </link> -->
+<link name="base">
+   <inertial>
+     <origin xyz="0 0 0" rpy="0 0 0"/>
+     <mass value="0.826"/>
+     <inertia ixx="1.205e-3"  ixy="0"  ixz="0" iyy="1.205e-3" iyz="0" izz="1.205e-3" />
+   </inertial>
+   <visual>
+     <origin xyz="0 0 0" rpy="0 0 0" />
+     <geometry>
+       <cylinder radius="0.05" length="0.1"/>
+     </geometry>
+     <material name="Cyan">
+       <color rgba="0 1.0 1.0 1.0"/>
+     </material>
+   </visual>
+   <collision>
+     <origin xyz="0 0 0" rpy="0 0 0"/>
+     <geometry>
+       <cylinder radius="0.05" length="0.1"/>
+     </geometry>
+   </collision>
+ </link>
+  <joint name="base_joint" type="fixed">
     <parent link="top_plate_link" />
+    <child link="base" />
+    <origin xyz="0 0 0.05" rpy="0 0 0" />
+  </joint>
+<!-- <joint name="bowler_joint" type="fixed">
+    <parent link="velodyne" />
     <child link="bowler_link" />
-    <origin xyz="0.1 -0.1 0" rpy="0 0 0.5" />
-  </joint>
+    <origin xyz="0 0 0" rpy="0 0 0.5" />
+</joint> -->
 </robot>

Commit message: Add files via upload

File: src/husky/urdf/teste.xacro (robot description, xacro)
@@ -4,8 +4,9 @@
   <xacro:property name="gpu" value="$(arg gpu)" />
   <!-- Insert customization below, sample provided: -->
-    <xacro:include filename="$(find velodyne_description)/urdf/VLP-16.urdf.xacro"/>
-    <VLP-16 parent="base" name="velodyne" topic="/velodyne_points" hz="10" samples="440" gpu="${gpu}">
+  <xacro:include filename="$(find velodyne_description)/urdf/VLP-16.urdf.xacro"/>
+  <VLP-16 parent="base" name="velodyne" topic="/velodyne_points" hz="10" samples="440" gpu="${gpu}">
     <origin xyz="0 0 0.1" rpy="0 0 0" />
   </VLP-16>
+  <xacro:include filename="$(find gazebo_light_sensor_plugin)/urdf/camera.xacro" />
  <!-- <link name="bowler_link">
     <visual>
@@ -53,3 +54,8 @@
     <origin xyz="0 0 0" rpy="0 0 0.5" />
 </joint> -->
+<joint name="camera_joint" type="fixed">
+    <parent link="top_plate_link" />
+    <child link="base_camera" />
+    <origin xyz="0.12 0 0.05" rpy="0 0 0" />
+</joint>
 </robot>
